File: KiCad/snes_rgb_bypass_amp.kicad_pcb (KiCad board)
At the start: 2 copper layers, 15.9 x 20.8 mm, 30 parts, among them U1 THS7374IPWR

Commit message: minor fix of bottom silk screen
Parts:
- moved *** 0.71 mm to (150.1, 110.1)
Changed lines of the file:
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@@
   )
   (module snes_rgb_bypass_amp:TM_logo-silk (layer B.Cu)
-    (at 149.63 109.5969 180)
+    (at 150.14 110.09 180)
     (descr "Made by TzorriMahm")
     (fp_text reference *** (at 0 4) (layer B.SilkS) hide
